File: clementina-hardware.kicad_pcb (KiCad board)
At the start: 2 copper layers, 172.7 x 108.6 mm, 48 parts, among them J1 Expansion, J2 Expansion, J3 User Port, J4 Audio Out, J5 microSD, SW1 RESET, U1 W65C02SxP, U2 AS6C4008-55PCN, U3 W65C22SxP, U4 AS6C62256-55PCN, U6 74HC138, U7 74HC08, U8 74HC138, U9 74HC04

Commit message: Board: re-route for the reworked glue logic
Same placement; U9 (now 74AC00) and U6's enables re-routed. DRC: no
errors, no unconnected items, no schematic parity issues (only the known
Pico library-mismatch warning). 122 vias, down from 137.

Co-Authored-By: Claude Opus 5.5 <noreply@anthropic.com>
Parts:
- U6, U8: value 74HC138 -> 74AC138
- U7: value 74HC08 -> 74AC08
- U9: value 74HC04 -> 74AC00
Connections:
- U6 pad 4: Net-(U6-~{E0}) -> /A13
- U6 pad 5: Net-(U6-~{E0}) -> /CS Logic/~{A15}
- U6 pad 6: +3.3V -> /A14
- U7 pad 4: /~{OE} -> GND
- U7 pad 5: /PHI2 -> GND
- U7 pad 6: Net-(U7-Pad6) -> unconnected-(U7-Pad6)
- U8 pad 13: Net-(U6-~{E0}) -> unconnected-(U8-~{Y2}-Pad13)
- U9 pad 10: /~{WE} -> Net-(U8-~{Y3})
- U9 pad 11: Net-(U7-Pad6) -> /CS Logic/~{A15}
- U9 pad 12: unconnected-(U9-Pad12) -> /A15
- U9 pad 13: GND -> /A15
- U9 pad 2: /~{OE} -> /RWB
- U9 pad 3: GND -> /~{OE}
- U9 pad 4: unconnected-(U9-Pad4) -> /~{OE}
- U9 pad 5: Net-(U8-~{Y3}) -> /PHI2
- U9 pad 6: /MIACS -> /~{WE}
- U9 pad 8: unconnected-(U9-Pad8) -> /MIACS
- U9 pad 9: GND -> Net-(U8-~{Y3})
Routing:
- net /A15: track 64.5 -> 123.6 mm, vias 3 -> 5
- net /CS Logic/~{A15}: track 0.00 -> 53.4 mm, vias 0 -> 1
- net /A13: track 104.5 -> 142.3 mm
- net /A14: track 77.7 -> 111.9 mm, vias 2 -> 4
- net Net-(U6-~{E0}): track 32.7 -> 0.00 mm, vias 2 -> 0
- net Net-(U7-Pad6): track 21.1 -> 0.00 mm, vias 1 -> 0
- net /D6: track 197.2 -> 217.7 mm
- net /A10: track 117.1 -> 135.0 mm, vias 3 -> 7
- net /A9: track 136.8 -> 154.5 mm, vias 2 -> 5
- net /~{WE}: track 165.4 -> 182.1 mm
- net /PHI2: track 200.7 -> 215.0 mm, vias 3 -> 2
- net /A12: track 104.0 -> 118.2 mm, vias 3 -> 4
- net Net-(U8-~{Y0}): track 66.9 -> 53.1 mm, vias 4 -> 0
- net /MIACS: track 162.3 -> 151.4 mm, vias 3 -> 1
- net /D7: track 206.6 -> 217.2 mm, vias 4 -> 3
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
Commit message: Tie the CPU's /SO to +3.3V
/SO (pin 38) had a no-connect flag. It is an input: a falling edge sets
the V flag, and WDC's datasheet requires unused input-only pins to be tied
to VDD, so a floating /SO could flip V at random (BVS/BVC after ADC, SBC,
BIT). It now goes to +3.3V like BE. The board is re-routed for the new
connection: DRC clean, no unconnected items, no parity issues.

Co-Authored-By: Claude Opus 5.5 <noreply@anthropic.com>
Connections:
- U1 pad 38: unconnected-(U1-~{SO}-Pad38) -> +3.3V
Routing:
- net /A10: track 135.0 -> 107.0 mm, vias 7 -> 3
- net /D7: track 217.2 -> 197.3 mm, vias 3 -> 2
- net /D5: track 188.1 -> 205.3 mm, vias 1 -> 6
- net /~{IRQB}: track 216.6 -> 201.8 mm, vias 0 -> 2
- net GND: track 609.8 -> 595.5 mm, vias 154 -> 151
- net /A8: track 145.9 -> 158.7 mm, vias 2 -> 5
- net /A6: track 130.4 -> 141.0 mm, vias 5 -> 4
- net /A9: track 154.5 -> 144.6 mm, vias 5 -> 2
- net /CB2: track 50.0 -> 40.1 mm, vias 0 -> 1
- net /A12: track 118.2 -> 109.4 mm
- net /MIACS: track 151.4 -> 159.4 mm
- net /RDY: track 124.4 -> 131.6 mm, vias 2 -> 3
- net /~{RESB}: track 225.1 -> 231.6 mm, vias 1 -> 5
- net /~{NMI}: track 139.1 -> 133.0 mm
- net /~{IOCS2}: track 44.2 -> 38.2 mm, vias 3 -> 2
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
Commit message: RDY pull-up: 1K -> 2.2K
RDY is bidirectional: the W65C02S pulls it low while it executes WAI, and
it only guarantees 1.6 mA at 0.4 V. Against 1K that would be ~2.9 mA and a
low level of roughly 0.65 V, out of spec. 2.2K keeps it at 1.5 mA. The
cost is a slower rise when a card releases RDY (~130 ns with ~50 pF),
harmless at the default 1.2 MHz and at most one extra wait state at 8 MHz.

The header note and README also warn card designers that RDY goes low
during WAI. Board: only R1's value changes (routing untouched).

Co-Authored-By: Claude Opus 5.5 <noreply@anthropic.com>
Parts:
- R1: value 1K -> 2.2K
Changed lines of the file:
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@@
 			)
 		)
-		(property "Value" "1K"
+		(property "Value" "2.2K"
 			(at 5.08 0 0)
 			(layer "F.SilkS")

Commit message: Clear the area past the Wi-Fi antenna
Raspberry Pi recommends the Pico W's antenna at a board edge with nothing
close to it. Moving it there would reshape the board, so for rev 1 the
nearest intrusions go instead:

- The reset button and its RC (R3, R4, C1) sat ~6 mm past the antenna's
  end; they move ~30 mm away, left of J1.
- A rule area ("Wi-Fi antenna clearance") on both layers keeps tracks,
  vias and GND fill ~6 mm past the Pico's end, extending the footprint's
  own antenna keep-out. The silkscreen says to keep it clear.

Re-routed: DRC clean, no unconnected items, no schematic parity issues.
The README explains the trade-off and how to check a build (RSSI with and
without the board; rev 2 moves the antenna to an edge if it costs > ~6 dB).

Co-Authored-By: Claude Opus 5.5 <noreply@anthropic.com>
Parts:
- moved SW1 26.7 mm to (69.2, 128.9)
- moved C1 26.7 mm to (89.5, 126.4)
- moved R3 26.7 mm to (81.9, 126.4)
- moved R4 26.7 mm to (85.7, 126.4)
Routing:
- net GND: track 595.5 -> 625.8 mm, vias 151 -> 146
- net +5V: track 212.4 -> 239.4 mm
- net /~{MIARESET}: track 49.0 -> 74.9 mm
- net /D4: track 188.8 -> 207.9 mm, vias 3 -> 1
- net /D7: track 197.3 -> 215.9 mm, vias 2 -> 4
- net /~{NMI}: track 133.0 -> 116.0 mm, vias 1 -> 4
- net /~{IRQB}: track 201.8 -> 217.3 mm
- net /D2: track 199.4 -> 213.2 mm, vias 4 -> 3
- net /MIACS: track 159.4 -> 146.5 mm, vias 1 -> 3
- net /A10: track 107.0 -> 116.9 mm, vias 3 -> 5
- net /A6: track 141.0 -> 131.1 mm, vias 4 -> 3
- net /RDY: track 131.6 -> 121.8 mm, vias 3 -> 0
- net /D5: track 205.3 -> 195.7 mm, vias 6 -> 5
- net /~{IOCS2}: track 38.2 -> 47.0 mm
- net /CB2: track 40.1 -> 48.8 mm, vias 1 -> 0
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Other:
- board text added: "Wi-Fi antenna: keep clear"
