File: CS Logic.kicad_sch (KiCad schematic)
At the start: 4 parts, among them U6 74HC138, U7 74LS08, U8 74HC138, U9 74HC04

Commit message: Rev 1 power section: run everything from the Pico's USB
- Pico 3V3 drives +3.3V, VBUS drives +5V for the header pins, and all
  GND pins plus AGND go to GND. VSYS is left free for a rev 2 power input.
  RUN, 3V3_EN, ADC_VREF and GP28 get no-connect flags.
- Decoupling: 100 nF per chip (C6-C13, each labelled with its chip) and
  22 uF bulk on +3.3V (C14).
- U5's only AND gate moves into U7's spare slot (U7B), and U5 is removed.
- U7 and U9 power units and spare gates are now on the sheet, with the
  spare gate inputs tied to GND so HC inputs don't float. U8's unused
  Y4-Y7 get no-connect flags.
- U7 74LS08 -> 74HC08, and U4 HM62256BLP -> AS6C62256-55PCN, because the
  LS08 and the HM62256 are 5 V-only parts.

Co-Authored-By: Claude Opus 5.5 <noreply@anthropic.com>
Parts:
- U7: value 74LS08 -> 74HC08
Connections:
- no-connect marks 0 -> 4
Changed lines of the file:
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@@
 		)
+	)
+	(no_connect
+		(at 99.06 68.58)
+	)
+	(no_connect
+		(at 99.06 71.12)
+	)
+	(no_connect
+		(at 99.06 73.66)
+	)
+	(no_connect
+		(at 99.06 76.2)
 	)
 	(symbol
@@
 			)
 		)
-		(property "Value" "74LS08"
+		(property "Value" "74HC08"
 			(at 129.5317 78.74 0)
 			(effects

Commit message: All through-hole parts: footprints, microSD breakout socket, round-pin jack
- Every part now has a through-hole footprint: DIP sockets for the chips,
  the Pico on 1x20 female headers (RaspberryPi_Pico_Common_THT), axial
  resistors and diodes, disc and radial capacitors, a 6 mm tactile switch.
- J5 is now a 1x9 female header for the Adafruit 4682 microSD breakout
  (3V, GND, CLK, SO, SI, CS, DAT1, DAT2, DET). The breakout has its own
  pull-ups and bypass caps, so RN1, C15 and C16 are gone. DAT1, DAT2 and
  DET are no-connects.
- J4 uses the CUI SJ1-3533NG footprint with round holes; the SJ1-3525N
  footprint needs 0.4 mm plated slots, below most hobby fabs' minimum.
- C3 and C5 (47 uF audio DC blocks) are drawn as polarized capacitors,
  + on the divider side.

Netlist unchanged apart from J5/RN1/C15/C16; ERC clean.

Co-Authored-By: Claude Opus 5.5 <noreply@anthropic.com>
Parts:
- U6, U8: footprint (none) -> Package_DIP:DIP-16_W7.62mm_Socket
- U7, U9: footprint (none) -> Package_DIP:DIP-14_W7.62mm_Socket
Changed lines of the file:
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@@
 			)
 		)
-		(property "Footprint" ""
+		(property "Footprint" "Package_DIP:DIP-14_W7.62mm_Socket"
 			(at 129.54 85.09 0)
 			(effects
@@
 			)
 		)
-		(property "Footprint" ""
+		(property "Footprint" "Package_DIP:DIP-16_W7.62mm_Socket"
 			(at 88.9 68.58 0)
 			(effects
@@
 			)
 		)
-		(property "Footprint" ""
+		(property "Footprint" "Package_DIP:DIP-16_W7.62mm_Socket"
 			(at 142.24 59.69 0)
 			(effects
@@
 			)
 		)
-		(property "Footprint" ""
+		(property "Footprint" "Package_DIP:DIP-14_W7.62mm_Socket"
 			(at 129.54 100.33 0)
 			(effects

Commit message: Glue logic: /WE from one NAND gate, flat I/O decode, 74AC parts
The write strobe went PHI2 -> 74HC08 -> 74HC04 -> /WE: about 26 ns typical
and up to ~65 ns at 3.3 V before /WE rose, against the W65C02S's 10 ns
address/data hold. With U4's /CE tied to A15, a store followed by an
access to another RAM address could also write that address.

- U9 is now a 74AC00 (quad NAND): ~OE = NAND(RWB, RWB),
  ~WE = NAND(PHI2, ~OE), MIASEL = NAND(~Y3, ~Y3), ~A15 = NAND(A15, A15).
  PHI2 reaches /WE through one gate (~5 ns typ, ~10 ns max as 74AC00),
  the same structure as the Picocomputer RP6502.
- U6 is enabled straight from the address (~E0 = A13, ~E1 = ~A15,
  E2 = A14) instead of through U8's ~Y2, removing one decoder level from
  the VIA/IOCS chip selects. U8 ~Y2 is now a no-connect.
- U7B becomes a spare (inputs to GND); U9's old spare inverters go.
- Values: U6/U8 74AC138, U7 74AC08, U9 74AC00 (all DIP).

The logic is unchanged (same truth tables). ERC clean.

Co-Authored-By: Claude Opus 5.5 <noreply@anthropic.com>
Parts:
- removed U9: 74HC04, Package_DIP:DIP-14_W7.62mm_Socket, symbol 74xx:74HC04
- added U9: 74AC00, Package_DIP:DIP-14_W7.62mm_Socket, symbol 74xx:74LS00
- U6, U8: value 74HC138 -> 74AC138
- U7: value 74HC08 -> 74AC08
Connections:
- net +3.3V: no longer U6.6 (E2)
- net A13: now also U6.4 (~{E0})
- net A14: now also U6.6 (E2)
- net A15: now also U9.12, U9.13
- net MIASEL: now also U9.8
- net at U8.12 (~{Y3}): now also U9.10, U9.9
- new net ~{A15}: U6.5 (~{E1}), U9.11
- now unconnected: U8.13 (~{Y2})
- no-connect marks 4 -> 5
Other:
- note added: "I/O slots ($C000-$DFFF): U6 is enabled straight from A13-A15 (one gate level) so the VIA and card chip selects settle early enough before PHI2 rises."

Commit message: Generic bill of materials for a solder-free build
Every part gets two hidden schematic fields:

- Factory: what is soldered at that designator, in generic terms (resistor
  value/size/pitch, capacitor type and lead spacing, DIP socket size for each
  chip, two 1x20 female headers for the Pico, box headers, jack, switch).
- Plug-in: what goes in afterwards (the chips, a Pico 2 WH with its pins
  pre-soldered, the Adafruit 4682).

bom/factory-bom.csv is generated from the Factory field with kicad-cli, so
the parts can be sourced by hand for the protoboard or given to an assembly
service. The README lists the plug-in parts and the regenerate command, and
notes that the 4682 ships with its header loose. Nets, ERC, DRC and parity
unchanged.

Co-Authored-By: Claude Opus 5.5 <noreply@anthropic.com>
Parts:
- U6, U8: Factory (none) -> DIP-16 socket, 7.62 mm (0.3 in) rows; Plug-in (none) -> 74AC138 3-to-8 decoder, DIP-16
- U7: Factory (none) -> DIP-14 socket, 7.62 mm (0.3 in) rows; Plug-in (none) -> 74AC08 quad AND, DIP-14
- U9: Factory (none) -> DIP-14 socket, 7.62 mm (0.3 in) rows; Plug-in (none) -> 74AC00 quad NAND, DIP-14
Changed lines of the file:
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@@
+			)
+		)
+		(property "Factory" "DIP-14 socket, 7.62 mm (0.3 in) rows"
+			(at 129.54 100.33 0)
+			(effects
+				(font
+					(size 1.27 1.27)
+				)
+				(hide yes)
+			)
+		)
+		(property "Plug-in" "74AC00 quad NAND, DIP-14"
+			(at 129.54 100.33 0)
+			(effects
+				(font
+					(size 1.27 1.27)
+				)
+				(hide yes)
 			)
 		)
@@
 		)
 		(property "Description" "quad 2-input NAND gate"
+			(at 129.54 115.57 0)
+			(effects
+				(font
+					(size 1.27 1.27)
+				)
+				(hide yes)
+			)
+		)
+		(property "Factory" "DIP-14 socket, 7.62 mm (0.3 in) rows"
+			(at 129.54 115.57 0)
+			(effects
+				(font
+					(size 1.27 1.27)
+				)
+				(hide yes)
+			)
+		)
+		(property "Plug-in" "74AC00 quad NAND, DIP-14"
 			(at 129.54 115.57 0)
 			(effects
@@
 			)
 		)
+		(property "Factory" "DIP-14 socket, 7.62 mm (0.3 in) rows"
+			(at 129.54 85.09 0)
+			(effects
+				(font
+					(size 1.27 1.27)
+				)
+				(hide yes)
+			)
+		)
+		(property "Plug-in" "74AC08 quad AND, DIP-14"
+			(at 129.54 85.09 0)
+			(effects
+				(font
+					(size 1.27 1.27)
+				)
+				(hide yes)
+			)
+		)
 		(pin "1"
 		)
@@
 			)
 		)
+		(property "Factory" "DIP-16 socket, 7.62 mm (0.3 in) rows"
+			(at 88.9 68.58 0)
+			(effects
+				(font
+					(size 1.27 1.27)
+				)
+				(hide yes)
+			)
+		)
+		(property "Plug-in" "74AC138 3-to-8 decoder, DIP-16"
+			(at 88.9 68.58 0)
+			(effects
+				(font
+					(size 1.27 1.27)
+				)
+				(hide yes)
+			)
+		)
 		(pin "13"
 		)
@@
 			(at 142.24 59.69 0)
 			(effects
+				(font
+					(size 1.27 1.27)
+				)
+				(hide yes)
+			)
+		)
+		(property "Factory" "DIP-16 socket, 7.62 mm (0.3 in) rows"
+			(at 142.24 59.69 0)
+			(effects
+				(font
+					(size 1.27 1.27)
+				)
+				(hide yes)
+			)
+		)
+		(property "Plug-in" "74AC138 3-to-8 decoder, DIP-16"
+			(at 142.24 59.69 0)
+			(effects
