File: clementina-hardware.kicad_sch (KiCad schematic)
At the start: 30 parts, among them J1 Expansion, J2 Expansion, J3 User Port, J4 Audio Out, SW1 RESET, U1 W65C02SxP, U2 AS6C4008-55PCN, U3 W65C22SxP, U4 HM62256BLP, U7 74LS08, U9 74HC04

Commit message: Rev 1 power section: run everything from the Pico's USB
- Pico 3V3 drives +3.3V, VBUS drives +5V for the header pins, and all
  GND pins plus AGND go to GND. VSYS is left free for a rev 2 power input.
  RUN, 3V3_EN, ADC_VREF and GP28 get no-connect flags.
- Decoupling: 100 nF per chip (C6-C13, each labelled with its chip) and
  22 uF bulk on +3.3V (C14).
- U5's only AND gate moves into U7's spare slot (U7B), and U5 is removed.
- U7 and U9 power units and spare gates are now on the sheet, with the
  spare gate inputs tied to GND so HC inputs don't float. U8's unused
  Y4-Y7 get no-connect flags.
- U7 74LS08 -> 74HC08, and U4 HM62256BLP -> AS6C62256-55PCN, because the
  LS08 and the HM62256 are 5 V-only parts.

Co-Authored-By: Claude Opus 5.5 <noreply@anthropic.com>
Parts:
- added C10, C11, C12, C13, C6, C7, C8, C9: 100nF, symbol Device:C
- added C14: 22uF, symbol Device:C_Polarized
- U4: value HM62256BLP -> AS6C62256-55PCN
- U7: value 74LS08 -> 74HC08
Connections:
- net +3.3V: now also A1.36 (3V3), U7.14 (VCC), U9.14 (VCC), C10.1, C11.1, C12.1, C13.1, C14.1, C6.1, C7.1, C8.1, C9.1
- net +5V: now also A1.40 (VBUS)
- net GND: now also A1.13 (GND), A1.18 (GND), A1.23 (GND), A1.28 (GND), A1.3 (GND), A1.33 (AGND), A1.38 (GND), A1.8 (GND), U7.10, U7.12, U7.13, U7.7 (GND), U7.9, U9.13, U9.3, U9.7 (GND), U9.9, C10.2, C11.2, C12.2, C13.2, C14.2, C6.2, C7.2, C8.2, C9.2
- no-connect marks 6 -> 16
Other:
- note added: "Decoupling: one 100 nF ceramic at each chip's VCC pin (chip named below); 22 uF bulk on +3.3V near the Pico's 3V3 pin. Rev 1 runs from the Pico's USB: keep the external 3V3 load under ~300 mA. VSYS is left free for a rev-2 power input."
- note added: "Pico"
- note added: "Spare gates: inputs tied to GND (HC inputs must not float). U7 and U9 power pins."
- note added: "U1"
- note added: "U2"
- note added: "U3"
- note added: "U4"
- note added: "U6"
- note added: "U7"
- note added: "U8"
- note added: "U9"
- moved on the sheet: U7C, U7D, U7E, U9B, U9D, U9F, U9G

Commit message: Add the microSD card and clear the remaining ERC items
- J5 microSD on MIA's SPI0 (GP0-GP3) in SPI mode. RN1 (4 x 10K bussed)
  pulls up CS, MISO, DAT1 and DAT2. C15 100 nF and C16 10 uF at the socket
  absorb insertion surges. A note covers building it with a 3V-only
  breakout on protoboard.
- PA5-PA7 get no-connect flags instead of dangling labels. W65C22S pins
  have bus-hold, so they don't float.
- U4 uses clementina:AS6C62256-55PCN from a new project library
  (clementina.kicad_sym + sym-lib-table), since KiCad 9 dropped
  HM62256BLP. The pinout is unchanged.
- The intentional AGND-GND join is recorded as a commented ERC exclusion
  in the project file. ERC is now clean.
- The header note says +5V comes from VBUS, that ~RESB is input-only for
  cards, and that W65C22S port pins have no current limiting.

Co-Authored-By: Claude Opus 5.5 <noreply@anthropic.com>
Parts:
- added C15: 100nF, symbol Device:C
- added C16: 10uF, symbol Device:C_Polarized
- added J5: microSD, Connector_Card:microSD_HC_Molex_47219-2001, symbol Connector:Micro_SD_Card
- added RN1: 10K, Resistor_THT:R_Array_SIP5, symbol Device:R_Network04
- U4: symbol Memory_RAM:HM62256BLP -> clementina:AS6C62256-55PCN
Connections:
- net +3.3V: now also C15.1, C16.1, J5.4 (VDD), RN1.1 (common)
- net GND: now also C15.2, C16.2, J5.6 (VSS), J5.9 (SHIELD)
- net SD_MISO: now reaches A1.1 (GPIO0)
- net SD_MISO: now also J5.7 (DAT0), RN1.3 (R2)
- net SD_CS: now reaches A1.2 (GPIO1)
- net SD_CS: now also J5.2 (DAT3/CD), RN1.4 (R3)
- net SD_SCK: now reaches A1.4 (GPIO2)
- net SD_SCK: now also J5.5 (CLK)
- net SD_MOSI: now reaches A1.5 (GPIO3)
- net SD_MOSI: now also J5.3 (CMD)
- net PA5: no longer names the net of U3.7 (PA5)
- net PA6: no longer names the net of U3.8 (PA6)
- net PA7: no longer names the net of U3.9 (PA7)
- new net SD_DAT1: J5.8 (DAT1), RN1.2 (R1)
- new net SD_DAT2: J5.1 (DAT2), RN1.5 (R4)
- no-connect marks 16 -> 19
Other:
- note added: "J1, J2 expansion bus / J3 user port (VIA port B) - 3.3 V logic only: no 5 V signals on any pin. - A card claims one I/O slot by jumpering one of ~{IOCS1}..~{IOCS7} ($C400-$DFFF, 1 KB each). - ~{IRQB}, ~{NMI} and RDY are wired-AND with pull-ups on this board: cards pull them low through a Schottky diode or an open-drain output, never drive them high. - ~{RESB} is driven by MIA: cards may read it b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"
- note added: "microSD in SPI mode on MIA's SPI0 (GP0-GP3): 400 kHz to initialise, then 12 MHz. RN1 keeps CS high while MIA boots and holds the lines the card leaves idle; C15/C16 absorb insertion surges. Protoboard: a 3V-only microSD breakout (e.g. Adafruit 4682) wired by signal name; skip parts the breakout already has."
- note removed: "J1, J2 expansion bus / J3 user port (VIA port B) - 3.3 V logic only: no 5 V signals on any pin. - A card claims one I/O slot by jumpering one of ~{IOCS1}..~{IOCS7} ($C400-$DFFF, 1 KB each). - ~{IRQB}, ~{NMI} and RDY are wired-AND with pull-ups on this board: cards pull them low through a Schottky diode or an open-drain output, never drive them high. - +5V pins have no source yet (power section TB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"

Commit message: All through-hole parts: footprints, microSD breakout socket, round-pin jack
- Every part now has a through-hole footprint: DIP sockets for the chips,
  the Pico on 1x20 female headers (RaspberryPi_Pico_Common_THT), axial
  resistors and diodes, disc and radial capacitors, a 6 mm tactile switch.
- J5 is now a 1x9 female header for the Adafruit 4682 microSD breakout
  (3V, GND, CLK, SO, SI, CS, DAT1, DAT2, DET). The breakout has its own
  pull-ups and bypass caps, so RN1, C15 and C16 are gone. DAT1, DAT2 and
  DET are no-connects.
- J4 uses the CUI SJ1-3533NG footprint with round holes; the SJ1-3525N
  footprint needs 0.4 mm plated slots, below most hobby fabs' minimum.
- C3 and C5 (47 uF audio DC blocks) are drawn as polarized capacitors,
  + on the divider side.

Netlist unchanged apart from J5/RN1/C15/C16; ERC clean.

Co-Authored-By: Claude Opus 5.5 <noreply@anthropic.com>
Parts:
- removed C15: 100nF, symbol Device:C
- removed C16: 10uF, symbol Device:C_Polarized
- removed J5: microSD, Connector_Card:microSD_HC_Molex_47219-2001, symbol Connector:Micro_SD_Card
- removed RN1: 10K, Resistor_THT:R_Array_SIP5, symbol Device:R_Network04
- added J5: microSD, Connector_PinSocket_2.54mm:PinSocket_1x09_P2.54mm_Vertical, symbol Connector:Conn_01x09_Socket
- A1: footprint Module:RaspberryPi_Pico_W_SMD_HandSolder -> Module:RaspberryPi_Pico_Common_THT
- C1, C10, C11, C12, C13, C2, C4, C6, C7, C8, C9: footprint (none) -> Capacitor_THT:C_Disc_D5.0mm_W2.5mm_P5.00mm
- C14: footprint (none) -> Capacitor_THT:CP_Radial_D5.0mm_P2.50mm
- C3, C5: footprint (none) -> Capacitor_THT:CP_Radial_D5.0mm_P2.50mm; symbol Device:C -> Device:C_Polarized
- D1, D2: footprint (none) -> Diode_THT:D_DO-34_SOD68_P7.62mm_Horizontal
- J4: footprint Connector_Audio:Jack_3.5mm_CUI_SJ1-3525N_Horizontal -> Connector_Audio:Jack_3.5mm_CUI_SJ1-3533NG_Horizontal_CircularHoles
- R1, R10, R11, R2, R3, R4, R5, R6, R7, R8, R9: footprint (none) -> Resistor_THT:R_Axial_DIN0207_L6.3mm_D2.5mm_P10.16mm_Horizontal
- SW1: footprint (none) -> Button_Switch_THT:SW_PUSH_6mm
- U1, U3: footprint Package_DIP:DIP-40_W15.24mm -> Package_DIP:DIP-40_W15.24mm_Socket
- U2: footprint Package_DIP:DIP-32_W15.24mm -> Package_DIP:DIP-32_W15.24mm_Socket
- U4: footprint Package_DIP:DIP-28_W15.24mm -> Package_DIP:DIP-28_W15.24mm_Socket
- U7, U9: footprint (none) -> Package_DIP:DIP-14_W7.62mm_Socket
Connections:
- net +3.3V: now also J5.1 (Pin_1)
- net GND: now also J5.2 (Pin_2)
- net SD_CS: now also J5.6 (Pin_6)
- net SD_MISO: now also J5.4 (Pin_4)
- net SD_MOSI: now also J5.5 (Pin_5)
- net SD_SCK: now also J5.3 (Pin_3)
- no-connect marks 19 -> 22
Other:
- note added: "3V"
- note added: "CLK"
- note added: "CS"
- note added: "DAT1"
- note added: "DAT2"
- note added: "DET"
- note added: "GND"
- note added: "SI"
- note added: "SO"
- note added: "microSD: J5 is a 9-pin female header for the Adafruit 4682 breakout (3V ONLY), in SPI mode on MIA's SPI0 (GP0-GP3): 400 kHz to initialise, then 12 MHz. The breakout has its own pull-ups on CS, MISO, DAT1, DAT2 and its own bypass caps. DAT1, DAT2 and DET stay unconnected. Use the same breakout on the protoboard build."
- note removed: "microSD in SPI mode on MIA's SPI0 (GP0-GP3): 400 kHz to initialise, then 12 MHz. RN1 keeps CS high while MIA boots and holds the lines the card leaves idle; C15/C16 absorb insertion surges. Protoboard: a 3V-only microSD breakout (e.g. Adafruit 4682) wired by signal name; skip parts the breakout already has."

Commit message: Glue logic: /WE from one NAND gate, flat I/O decode, 74AC parts
The write strobe went PHI2 -> 74HC08 -> 74HC04 -> /WE: about 26 ns typical
and up to ~65 ns at 3.3 V before /WE rose, against the W65C02S's 10 ns
address/data hold. With U4's /CE tied to A15, a store followed by an
access to another RAM address could also write that address.

- U9 is now a 74AC00 (quad NAND): ~OE = NAND(RWB, RWB),
  ~WE = NAND(PHI2, ~OE), MIASEL = NAND(~Y3, ~Y3), ~A15 = NAND(A15, A15).
  PHI2 reaches /WE through one gate (~5 ns typ, ~10 ns max as 74AC00),
  the same structure as the Picocomputer RP6502.
- U6 is enabled straight from the address (~E0 = A13, ~E1 = ~A15,
  E2 = A14) instead of through U8's ~Y2, removing one decoder level from
  the VIA/IOCS chip selects. U8 ~Y2 is now a no-connect.
- U7B becomes a spare (inputs to GND); U9's old spare inverters go.
- Values: U6/U8 74AC138, U7 74AC08, U9 74AC00 (all DIP).

The logic is unchanged (same truth tables). ERC clean.

Co-Authored-By: Claude Opus 5.5 <noreply@anthropic.com>
Parts:
- removed U9: 74HC04, Package_DIP:DIP-14_W7.62mm_Socket, symbol 74xx:74HC04
- added unit 2 of U7
- added U9: 74AC00, Package_DIP:DIP-14_W7.62mm_Socket, symbol 74xx:74LS00
- U7: value 74HC08 -> 74AC08
Connections:
- net +3.3V: now also U9.14 (VCC)
- net GND: now also U7.4, U7.5, U9.7 (GND)
- no-connect marks 22 -> 20
Other:
- note added: "Spare gates: inputs tied to GND (CMOS inputs must not float). U7 and U9 power pins."
- note removed: "Spare gates: inputs tied to GND (HC inputs must not float). U7 and U9 power pins."

Commit message: Tie the CPU's /SO to +3.3V
/SO (pin 38) had a no-connect flag. It is an input: a falling edge sets
the V flag, and WDC's datasheet requires unused input-only pins to be tied
to VDD, so a floating /SO could flip V at random (BVS/BVC after ADC, SBC,
BIT). It now goes to +3.3V like BE. The board is re-routed for the new
connection: DRC clean, no unconnected items, no parity issues.

Co-Authored-By: Claude Opus 5.5 <noreply@anthropic.com>
Connections:
- net +3.3V: now also U1.38 (~{SO})
- no-connect marks 20 -> 19
Changed lines of the file:
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@@
 	)
 	(no_connect
-		(at 27.94 167.64)
-	)
-	(no_connect
 		(at 27.94 129.54)
 	)
@@
 		)
 	)
+	(wire
+		(pts
+			(xy 27.94 167.64) (xy 25.4 167.64)
+		)
+		(stroke
+			(width 0)
+			(type default)
+		)
+	)
+	(symbol
+		(lib_id "power:+3.3V")
+		(at 25.4 167.64 90)
+		(unit 1)
+		(exclude_from_sim no)
+		(in_bom no)
+		(on_board yes)
+		(dnp no)
+		(property "Reference" "#PWR083"
+			(at 25.4 167.64 90)
+			(effects
+				(font
+					(size 1.27 1.27)
+				)
+				(hide yes)
+			)
+		)
+		(property "Value" "+3.3V"
+			(at 19.1 167.64 90)
+			(effects
+				(font
+					(size 1.27 1.27)
+				)
+			)
+		)
+		(property "Footprint" ""
+			(at 25.4 167.64 0)
+			(effects
+				(font
+					(size 1.27 1.27)
+				)
+				(hide yes)
+			)
+		)
+		(property "Datasheet" ""
+			(at 25.4 167.64 0)
+			(effects
+				(font
+					(size 1.27 1.27)
+				)
+				(hide yes)
+			)
+		)
+		(property "Description" "Power symbol creates a global label with name \"+3.3V\""
+			(at 25.4 167.64 0)
+			(effects
+				(font
+					(size 1.27 1.27)
+				)
+				(hide yes)
+			)
+		)
+		(pin "1"
+		)
+		(instances
+			(project ""
+				(path "/ddb0bb09-4973-4322-81e7-cdd57ff08282"
+					(reference "#PWR083")
+					(unit 1)
+				)
+			)
+		)
+	)

Commit message: RDY pull-up: 1K -> 2.2K
RDY is bidirectional: the W65C02S pulls it low while it executes WAI, and
it only guarantees 1.6 mA at 0.4 V. Against 1K that would be ~2.9 mA and a
low level of roughly 0.65 V, out of spec. 2.2K keeps it at 1.5 mA. The
cost is a slower rise when a card releases RDY (~130 ns with ~50 pF),
harmless at the default 1.2 MHz and at most one extra wait state at 8 MHz.

The header note and README also warn card designers that RDY goes low
during WAI. Board: only R1's value changes (routing untouched).

Co-Authored-By: Claude Opus 5.5 <noreply@anthropic.com>
Parts:
- R1: value 1K -> 2.2K
Other:
- note added: "J1, J2 expansion bus / J3 user port (VIA port B) - 3.3 V logic only: no 5 V signals on any pin. - A card claims one I/O slot by jumpering one of ~{IOCS1}..~{IOCS7} ($C400-$DFFF, 1 KB each). - ~{IRQB}, ~{NMI} and RDY are wired-AND with pull-ups on this board: cards pull them low through a Schottky diode or an open-drain output, never drive them high. - RDY also goes low while the CPU executes WAI.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"
- note removed: "J1, J2 expansion bus / J3 user port (VIA port B) - 3.3 V logic only: no 5 V signals on any pin. - A card claims one I/O slot by jumpering one of ~{IOCS1}..~{IOCS7} ($C400-$DFFF, 1 KB each). - ~{IRQB}, ~{NMI} and RDY are wired-AND with pull-ups on this board: cards pull them low through a Schottky diode or an open-drain output, never drive them high. - ~{RESB} is driven by MIA: cards may read it b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"
Changed lines of the file:
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@@
 			)
 		)
-		(property "Value" "1K"
+		(property "Value" "2.2K"
 			(at 26.67 71.755 90)
 			(effects
@@
 		)
 	)
-	(text "J1, J2 expansion bus / J3 user port (VIA port B)\n- 3.3 V logic only: no 5 V signals on any pin.\n- A card claims one I/O slot by jumpering one of\n  ~{IOCS1}..~{IOCS7} ($C400-$DFFF, 1 KB each).\n- ~{IRQB}, ~{NMI} and RDY are wired-AND with pull-ups\n  on this board: cards pull them low through a Schottky\n  diode or an open-drain output, never drive them high.\n- ~{RESB} is driven by MIA: cards may read it but\n  must never drive it.\n- +5V pins come from the Pico's VBUS (USB 5 V)\n  in rev 1.\n- W65C22S port pins have no current limiting: drive\n  LEDs and similar loads through a resistor."
+	(text "J1, J2 expansion bus / J3 user port (VIA port B)\n- 3.3 V logic only: no 5 V signals on any pin.\n- A card claims one I/O slot by jumpering one of\n  ~{IOCS1}..~{IOCS7} ($C400-$DFFF, 1 KB each).\n- ~{IRQB}, ~{NMI} and RDY are wired-AND with pull-ups\n  on this board: cards pull them low through a Schottky\n  diode or an open-drain output, never drive them high.\n- RDY also goes low while the CPU executes WAI.\n- ~{RESB} is driven by MIA: cards may read it but\n  must never drive it.\n- +5V pins come from the Pico's VBUS (USB 5 V)\n  in rev 1.\n- W65C22S port pins have no current limiting: drive\n  LEDs and similar loads through a resistor."
 		(exclude_from_sim no)
 		(at 350.52 99.06 0)

Commit message: Generic bill of materials for a solder-free build
Every part gets two hidden schematic fields:

- Factory: what is soldered at that designator, in generic terms (resistor
  value/size/pitch, capacitor type and lead spacing, DIP socket size for each
  chip, two 1x20 female headers for the Pico, box headers, jack, switch).
- Plug-in: what goes in afterwards (the chips, a Pico 2 WH with its pins
  pre-soldered, the Adafruit 4682).

bom/factory-bom.csv is generated from the Factory field with kicad-cli, so
the parts can be sourced by hand for the protoboard or given to an assembly
service. The README lists the plug-in parts and the regenerate command, and
notes that the 4682 ships with its header loose. Nets, ERC, DRC and parity
unchanged.

Co-Authored-By: Claude Opus 5.5 <noreply@anthropic.com>
Parts:
- A1: Factory (none) -> 2 x female header 1x20, 2.54 mm, 8.5 mm tall (both at A1, o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; Plug-in (none) -> Raspberry Pi Pico 2 WH (pins pre-soldered)
- C1: Factory (none) -> Ceramic capacitor 1 µF, 50 V, X7R, radial, 5.08 mm lead spa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
- C10, C11, C12, C13, C2, C4, C6, C7, C8, C9: Factory (none) -> Ceramic capacitor 100 nF, 50 V, X7R, radial, 5.08 mm lead s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
- C14: Factory (none) -> Electrolytic capacitor 22 µF, 16 V, radial, 5 mm diameter, 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
- C3, C5: Factory (none) -> Electrolytic capacitor 47 µF, 16 V, radial, 5 mm diameter, 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
- D1, D2: Factory (none) -> BAT85 Schottky diode, DO-34
- J1, J2: Factory (none) -> IDC box header 2x20, 2.54 mm, vertical
- J3: Factory (none) -> IDC box header 2x10, 2.54 mm, vertical
- J4: Factory (none) -> 3.5 mm stereo jack, CUI SJ1-3533NG or same footprint
- J5: Factory (none) -> Female header 1x9, 2.54 mm, 8.5 mm tall; Plug-in (none) -> Adafruit 4682 microSD breakout, 3 V (solder its header)
- R1: Factory (none) -> Resistor 2.2 kΩ, 1/4 W, 1% metal film, axial, 10.16 mm lead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
- R10, R4, R7: Factory (none) -> Resistor 100 Ω, 1/4 W, 1% metal film, axial, 10.16 mm lead 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
- R11, R8: Factory (none) -> Resistor 1.8 kΩ, 1/4 W, 1% metal film, axial, 10.16 mm lead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
- R2, R5: Factory (none) -> Resistor 4.7 kΩ, 1/4 W, 1% metal film, axial, 10.16 mm lead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
- R3: Factory (none) -> Resistor 10 kΩ, 1/4 W, 1% metal film, axial, 10.16 mm lead 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
- R6, R9: Factory (none) -> Resistor 220 Ω, 1/4 W, 1% metal film, axial, 10.16 mm lead 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
- SW1: Factory (none) -> Tactile switch 6 x 6 mm, through-hole
- U1: Factory (none) -> DIP-40 socket, 15.24 mm (0.6 in) rows; Plug-in (none) -> WDC W65C02S CPU, DIP-40 (W65C02S6TPG-14)
- U2: Factory (none) -> DIP-32 socket, 15.24 mm (0.6 in) rows; Plug-in (none) -> Alliance AS6C4008-55PCN 512K x 8 SRAM, DIP-32
- U3: Factory (none) -> DIP-40 socket, 15.24 mm (0.6 in) rows; Plug-in (none) -> WDC W65C22S VIA, DIP-40 (W65C22S6TPG-14)
- U4: Factory (none) -> DIP-28 socket, 15.24 mm (0.6 in) rows; Plug-in (none) -> Alliance AS6C62256-55PCN 32K x 8 SRAM, DIP-28
- U7: Factory (none) -> DIP-14 socket, 7.62 mm (0.3 in) rows; Plug-in (none) -> 74AC08 quad AND, DIP-14
- U9: Factory (none) -> DIP-14 socket, 7.62 mm (0.3 in) rows; Plug-in (none) -> 74AC00 quad NAND, DIP-14
